Commit message: vision based navigation

File: urdf/ict_bot.urdf (robot description, URDF)
Before this commit: robot ict_bot, 6 links, 5 joints
Links:
- added link camera_link, mass 0.05; collision box size=0.025 0.090 0.025; visual box size=0.025 0.090 0.025
- added link camera_optical_link
Joints:
- added joint camera_joint: type fixed, parent link_base, child camera_link, origin xyz=0 -0.08 0.10 rpy=0 0 -1.5708
- added joint camera_optical_joint: type fixed, parent camera_link, child camera_optical_link, origin xyz=0 0 0 rpy=-1.5708 0 -1.5708

Commit message: navigation in ofc environment

File: urdf/ict_bot.urdf (robot description, URDF)
Before this commit: robot ict_bot, 6 links, 5 joints
Links:
- added link lidar_3d, mass 0.1; collision cylinder length=0.06 radius=0.04; visual cylinder length=0.06 radius=0.04
Joints:
- added joint lidar_3d_joint: type fixed, parent link_base, child lidar_3d, origin xyz=0 -0.0284286 0.22 rpy=0 0 0
